Commit message: Add perception calibration helper and integrate aruco with calibration

File: src/dobot_rviz/urdf/cr10_robot.urdf (robot description, URDF)
Before this commit: robot cr10_robot, 8 links, 7 joints
Links:
- added link camera_link
Joints:
- added joint camera_mount: type fixed, parent Link6, child camera_link, origin xyz=0 -0.074 -0.03 rpy=-0.174533 0 0

File: src/dobot_rviz/urdf/cr12_robot.urdf (robot description, URDF)
Before this commit: robot cr12_robot, 8 links, 7 joints
Links:
- added link camera_link
Joints:
- added joint camera_mount: type fixed, parent Link6, child camera_link, origin xyz=0 -0.074 -0.03 rpy=-0.174533 0 0

File: src/dobot_rviz/urdf/cr16_robot.urdf (robot description, URDF)
Before this commit: robot cr16_robot, 8 links, 7 joints
Links:
- added link camera_link
Joints:
- added joint camera_mount: type fixed, parent Link6, child camera_link, origin xyz=0 -0.074 -0.03 rpy=-0.174533 0 0

File: src/dobot_rviz/urdf/cr20_robot.urdf (robot description, URDF)
Before this commit: robot cr20_robot, 8 links, 7 joints
Links:
- added link camera_link
Joints:
- added joint camera_mount: type fixed, parent Link6, child camera_link, origin xyz=0 -0.074 -0.03 rpy=-0.174533 0 0

File: src/dobot_rviz/urdf/cr30h_robot.urdf (robot description, URDF)
Before this commit: robot cr30h_robot, 8 links, 7 joints
Links:
- added link camera_link
Joints:
- added joint camera_mount: type fixed, parent Link6, child camera_link, origin xyz=0 -0.074 -0.03 rpy=-0.174533 0 0

File: src/dobot_rviz/urdf/cr3_robot.urdf (robot description, URDF)
Before this commit: robot cr3_robot, 8 links, 7 joints
Links:
- added link camera_link
Joints:
- added joint camera_mount: type fixed, parent Link6, child camera_link, origin xyz=0 -0.074 -0.03 rpy=-0.174533 0 0

File: src/dobot_rviz/urdf/cr5_robot.urdf (robot description, URDF)
Before this commit: robot cr5_robot, 8 links, 7 joints
Links:
- added link camera_link
Joints:
- added joint camera_mount: type fixed, parent Link6, child camera_link, origin xyz=0 -0.074 -0.03 rpy=-0.174533 0 0

File: src/dobot_rviz/urdf/cr7_robot.urdf (robot description, URDF)
Before this commit: robot cr7_robot, 8 links, 7 joints
Links:
- added link camera_link
Joints:
- added joint camera_mount: type fixed, parent Link6, child camera_link, origin xyz=0 -0.074 -0.03 rpy=-0.174533 0 0

File: src/dobot_rviz/urdf/me6_robot.urdf (robot description, URDF)
Before this commit: robot me6_robot, 8 links, 7 joints
Links:
- added link camera_link
Joints:
- added joint camera_mount: type fixed, parent Link6, child camera_link, origin xyz=0 -0.074 -0.03 rpy=-0.174533 0 0

File: src/dobot_rviz/urdf/nova2_robot.urdf (robot description, URDF)
Before this commit: robot nova2_robot, 8 links, 7 joints
Links:
- added link camera_link
Joints:
- added joint camera_mount: type fixed, parent Link6, child camera_link, origin xyz=0 -0.074 -0.03 rpy=-0.174533 0 0

File: src/dobot_rviz/urdf/nova5_robot.urdf (robot description, URDF)
Before this commit: robot nova5_robot, 7 links, 6 joints
Links:
- added link camera_link
Joints:
- added joint camera_mount: type fixed, parent Link6, child camera_link, origin xyz=0 -0.074 -0.03 rpy=-0.174533 0 0
